File: PCB/8266_DIYIOT_Board_C/8266_DIYIOT_Board_C_G_V_AS.sch (EAGLE design)
At the start: 16 parts

Commit message: lots of updates
Parts:
- added R1, R2: (no value), eagle-ltspice:R0204/7
Connections:
- removed net N$3: SIGNAL.P, U$4.ADC
- new net N$2: R1.2, SIGNAL.P
- new net N$4: R1.1, R2.2, U$4.ADC
- net 5V: now also R2.1
Changed lines of the file:
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@@
 <layer number="97" name="Info" color="7" fill="1" visible="yes" active="yes"/>
 <layer number="98" name="Guide" color="6" fill="1" visible="yes" active="yes"/>
+<layer number="99" name="SpiceOrder" color="5" fill="1" visible="yes" active="yes"/>
 <layer number="101" name="Hidden" color="15" fill="1" visible="yes" active="yes"/>
 <layer number="102" name="Changes" color="12" fill="1" visible="yes" active="yes"/>
@@
 <part name="5V_PIR" library="wirepad" deviceset="2,15/1,0" device=""/>
 <part name="SIGNAL" library="wirepad" deviceset="2,15/1,0" device=""/>
+<part name="R1" library="eagle-ltspice" deviceset="R" device="0204/7"/>
+<part name="R2" library="eagle-ltspice" deviceset="R" device="0204/7"/>
 </parts>
 <sheets>
@@
 <instance part="5V_PIR" gate="1" x="76.2" y="91.44"/>
 <instance part="SIGNAL" gate="1" x="86.36" y="83.82"/>
+<instance part="R1" gate="G$1" x="78.74" y="78.74"/>
+<instance part="R2" gate="G$1" x="63.5" y="78.74"/>
 </instances>
 <busses>
@@
 <pinref part="GND_1" gate="1" pin="P"/>
 <pinref part="GND_PIR" gate="1" pin="P"/>
+<pinref part="R2" gate="G$1" pin="1"/>
+<wire x1="58.42" y1="78.74" x2="58.42" y2="20.32" width="0.1524" layer="91"/>
+<wire x1="58.42" y1="20.32" x2="137.16" y2="20.32" width="0.1524" layer="91"/>
+<wire x1="137.16" y1="20.32" x2="139.7" y2="22.86" width="0.1524" layer="91"/>
+<wire x1="139.7" y1="22.86" x2="139.7" y2="38.1" width="0.1524" layer="91"/>
+<junction x="139.7" y="38.1"/>
 </segment>
 <segment>
@@
 </segment>
 </net>
-<net name="N$3" class="0">
+<net name="N$2" class="0">
 <segment>
 <pinref part="SIGNAL" gate="1" pin="P"/>
-<wire x1="66.04" y1="71.12" x2="88.9" y2="71.12" width="0.1524" layer="91"/>
-<wire x1="88.9" y1="71.12" x2="88.9" y2="83.82" width="0.1524" layer="91"/>
-<wire x1="66.04" y1="71.12" x2="66.04" y2="53.34" width="0.1524" layer="91"/>
+<wire x1="88.9" y1="83.82" x2="88.9" y2="78.74" width="0.1524" layer="91"/>
+<pinref part="R1" gate="G$1" pin="2"/>
+<wire x1="88.9" y1="78.74" x2="83.82" y2="78.74" width="0.1524" layer="91"/>
+<junction x="83.82" y="78.74"/>
+</segment>
+</net>
+<net name="N$4" class="0">
+<segment>
 <wire x1="76.2" y1="53.34" x2="73.66" y2="53.34" width="0.1524" layer="91"/>
 <pinref part="U$4" gate="G$1" pin="ADC"/>
-<wire x1="66.04" y1="53.34" x2="73.66" y2="53.34" width="0.1524" layer="91"/>
+<wire x1="68.58" y1="78.74" x2="68.58" y2="53.34" width="0.1524" layer="91"/>
+<wire x1="68.58" y1="53.34" x2="73.66" y2="53.34" width="0.1524" layer="91"/>
+<pinref part="R1" gate="G$1" pin="1"/>
+<junction x="68.58" y="78.74"/>
+<pinref part="R2" gate="G$1" pin="2"/>
+<wire x1="68.58" y1="78.74" x2="73.66" y2="78.74" width="0.1524" layer="91"/>
 </segment>
 </net>
