File: PCB/8266_DIYIOT_Board_F/8266_DIYIOT_Board_F_AS_V_G.brd (EAGLE design)
At the start: 70.8 x 74.9 mm, 20 parts

Commit message: lots of updates
Parts:
- added R1, R2: (no value), eagle-ltspice:0204/7
Connections:
- new net N$2: R1.2, SIGNAL.1
- net 5V: now also R2.1
- net N$3: now also R1.1, R2.2; no longer SIGNAL.1
Routing:
- net 5V: track 296.5 -> 333.7 mm
- net N$3: track 33.2 -> 20.4 mm
- net N$2: track 0.00 -> 11.9 mm
Changed lines of the file:
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@@
 <layer number="97" name="Info" color="7" fill="1" visible="no" active="no"/>
 <layer number="98" name="Guide" color="6" fill="1" visible="no" active="no"/>
+<layer number="99" name="SpiceOrder" color="5" fill="1" visible="no" active="no"/>
 <layer number="101" name="Hidden" color="15" fill="1" visible="yes" active="yes"/>
 <layer number="102" name="Changes" color="12" fill="1" visible="yes" active="yes"/>
@@
 <attribute name="VALUE" x="59.69" y="74.66" size="0.0254" layer="27"/>
 </element>
+<element name="R1" library="eagle-ltspice" package="0204/7" value="" x="49.53" y="66.04">
+<attribute name="SPICEMODEL" value="NONE" x="49.53" y="66.04" size="1.778" layer="27" display="off"/>
+<attribute name="SPICEPREFIX" value="R" x="49.53" y="66.04" size="1.778" layer="27" display="off"/>
+</element>
+<element name="R2" library="eagle-ltspice" package="0204/7" value="" x="38.1" y="66.04">
+<attribute name="SPICEMODEL" value="NONE" x="38.1" y="66.04" size="1.778" layer="27" display="off"/>
+<attribute name="SPICEPREFIX" value="R" x="38.1" y="66.04" size="1.778" layer="27" display="off"/>
+</element>
 </elements>
 <signals>
@@
 <wire x1="67.31" y1="20.32" x2="33.02" y2="20.32" width="0.4064" layer="16"/>
 <wire x1="33.02" y1="20.32" x2="27.94" y2="26.67" width="0.4064" layer="16"/>
-<wire x1="27.94" y1="26.67" x2="27.94" y2="46.99" width="0.4064" layer="16"/>
-<wire x1="27.94" y1="46.99" x2="36.89865" y2="63.088109375" width="0.4064" layer="16"/>
+<wire x1="27.94" y1="26.67" x2="27.94" y2="58.42" width="0.4064" layer="16"/>
+<wire x1="27.94" y1="58.42" x2="33.08865" y2="70.708109375" width="0.4064" layer="16"/>
 <contactref element="GND_PIR" pad="1"/>
 <contactref element="5V_PIR" pad="1"/>
-<wire x1="36.89865" y1="63.088109375" x2="50.8" y2="66.04" width="0.4064" layer="16"/>
-<wire x1="57.15" y1="73.66" x2="50.8" y2="66.04" width="0.4064" layer="16"/>
+<wire x1="33.08865" y1="70.708109375" x2="54.61" y2="71.12" width="0.4064" layer="16"/>
+<wire x1="57.15" y1="73.66" x2="54.61" y2="71.12" width="0.4064" layer="16"/>
 <wire x1="54.61" y1="73.66" x2="58.42" y2="77.47" width="0.4064" layer="16"/>
+<contactref element="R2" pad="1"/>
+<wire x1="34.29" y1="66.04" x2="30.48" y2="55.88" width="0.4064" layer="16"/>
+<wire x1="30.48" y1="55.88" x2="30.48" y2="36.83" width="0.4064" layer="16"/>
 <wire x1="74.93" y1="22.86" x2="74.93" y2="24.13" width="0" layer="19" extent="16-16"/>
 </signal>
@@
 </signal>
 <signal name="N$3">
-<contactref element="SIGNAL" pad="1"/>
-<wire x1="59.69" y1="73.66" x2="54.61" y2="66.04" width="0.4064" layer="16"/>
-<wire x1="54.61" y1="66.04" x2="43.18" y2="59.69" width="0.4064" layer="16"/>
-<wire x1="43.18" y1="59.69" x2="43.18" y2="54.61" width="0.4064" layer="16"/>
-<wire x1="46.84" y1="43.33" x2="43.18" y2="54.61" width="0" layer="19" extent="1-16"/>
 <contactref element="U$4" pad="ADC"/>
 <wire x1="48.78" y1="53.33" x2="45.72" y2="53.33" width="0.4064" layer="16"/>
-<wire x1="45.72" y1="53.33" x2="43.18" y2="54.61" width="0.4064" layer="16"/>
+<contactref element="R1" pad="1"/>
+<contactref element="R2" pad="2"/>
+<wire x1="45.72" y1="66.04" x2="41.91" y2="66.04" width="0.4064" layer="16"/>
+<wire x1="41.91" y1="66.04" x2="44.45" y2="54.6" width="0.4064" layer="16"/>
+<wire x1="44.45" y1="54.6" x2="45.72" y2="53.33" width="0.4064" layer="16"/>
+</signal>
+<signal name="N$2">
+<contactref element="SIGNAL" pad="1"/>
+<contactref element="R1" pad="2"/>
+<wire x1="59.69" y1="73.66" x2="59.69" y2="68.58" width="0.4064" layer="16"/>
+<wire x1="59.69" y1="68.58" x2="53.34" y2="66.04" width="0.4064" layer="16"/>
 </signal>
 </signals>
