File: PCB/8266_DIYIOT_Board_K/8266_DIYIOT_Board_K_G_V_SDA_SCL.brd (EAGLE design)
At the start: 70.8 x 74.9 mm, 21 parts

Commit message: lots of updates
Other:
- board text added: "DIYIOT - Board K"
- board text removed: "DIYIOT - Board D"
Changed lines of the file:
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@@
 <text x="55.88" y="76.2" size="1.778" layer="25">V</text>
 <text x="64.77" y="76.2" size="1.778" layer="25">SCL</text>
-<text x="24.13" y="49.53" size="1.778" layer="25" rot="R90">DIYIOT - Board D</text>
+<text x="24.13" y="49.53" size="1.778" layer="25" rot="R90">DIYIOT - Board K</text>
 <text x="58.42" y="76.2" size="1.778" layer="25">SDA</text>
 </plain>
