File: PCB/8266_DIYIOT_Board_O/Knob_8266.brd (EAGLE design)
At the start: 70.8 x 74.9 mm, 20 parts

Commit message: lots of updates
Parts:
- added 1K, 2K: (no value), eagle-ltspice:0204/7
Connections:
- new net N$3: 2K.2, POT_SIGNAL.1
- net 5V: now also 1K.2
- net N$2: now also 1K.1, 2K.1; no longer POT_SIGNAL.1
Routing:
- net 5V: track 287.6 -> 300.4 mm
- net N$2: track 37.2 -> 46.3 mm
- net N$3: track 0.00 -> 6.13 mm
Changed lines of the file:
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@@
 <layer number="97" name="Info" color="7" fill="1" visible="no" active="no"/>
 <layer number="98" name="Guide" color="6" fill="1" visible="no" active="no"/>
+<layer number="99" name="SpiceOrder" color="5" fill="1" visible="no" active="no"/>
 <layer number="101" name="Hidden" color="15" fill="1" visible="yes" active="yes"/>
 <layer number="102" name="Changes" color="12" fill="1" visible="yes" active="yes"/>
@@
 <attribute name="VALUE" x="52.07" y="77.2" size="0.0254" layer="27"/>
 </element>
+<element name="2K" library="eagle-ltspice" package="0204/7" value="" x="50.8" y="71.12" smashed="yes">
+<attribute name="SPICEMODEL" value="NONE" x="50.8" y="71.12" size="1.778" layer="27" display="off"/>
+<attribute name="SPICEPREFIX" value="R" x="50.8" y="71.12" size="1.778" layer="27" display="off"/>
+<attribute name="NAME" x="48.26" y="72.4154" size="0.9906" layer="25" ratio="10"/>
+<attribute name="VALUE" x="49.1744" y="70.6374" size="0.9906" layer="27" ratio="10"/>
+</element>
+<element name="1K" library="eagle-ltspice" package="0204/7" value="" x="63.5" y="68.58" smashed="yes">
+<attribute name="SPICEMODEL" value="NONE" x="63.5" y="68.58" size="1.778" layer="27" display="off"/>
+<attribute name="SPICEPREFIX" value="R" x="63.5" y="68.58" size="1.778" layer="27" display="off"/>
+<attribute name="NAME" x="60.96" y="69.8754" size="0.9906" layer="25" ratio="10"/>
+<attribute name="VALUE" x="61.8744" y="68.0974" size="0.9906" layer="27" ratio="10"/>
+</element>
 </elements>
 <signals>
@@
 <wire x1="52.07" y1="76.2" x2="48.26" y2="76.2" width="0.4064" layer="16"/>
 <wire x1="62.23" y1="76.2" x2="67.31" y2="76.2" width="0.4064" layer="16"/>
+<contactref element="1K" pad="2"/>
 <wire x1="74.93" y1="22.86" x2="74.93" y2="24.13" width="0" layer="19" extent="16-16"/>
+<wire x1="67.31" y1="68.58" x2="71.12" y2="68.58" width="0.4064" layer="16"/>
+<wire x1="71.12" y1="68.58" x2="77.47" y2="62.23" width="0.4064" layer="16"/>
+<wire x1="77.47" y1="62.23" x2="76.2" y2="62.23" width="0" layer="19" extent="1-16"/>
 </signal>
 <signal name="TX">
@@
 <signal name="N$2">
 <contactref element="U$4" pad="ADC"/>
-<contactref element="POT_SIGNAL" pad="1"/>
-<wire x1="48.78" y1="53.33" x2="45.73" y2="53.33" width="0.4064" layer="16"/>
-<wire x1="45.73" y1="53.33" x2="41.91" y2="57.15" width="0.4064" layer="16"/>
-<wire x1="41.91" y1="57.15" x2="41.91" y2="66.04" width="0.4064" layer="16"/>
-<wire x1="41.91" y1="66.04" x2="43.18" y2="67.31" width="0.4064" layer="16"/>
-<wire x1="43.18" y1="67.31" x2="49.53" y2="67.31" width="0.4064" layer="16"/>
-<wire x1="49.53" y1="67.31" x2="57.15" y2="76.2" width="0.4064" layer="16"/>
+<contactref element="2K" pad="1"/>
+<wire x1="46.99" y1="71.12" x2="43.18" y2="71.12" width="0.4064" layer="16"/>
+<wire x1="43.18" y1="71.12" x2="40.64" y2="68.58" width="0.4064" layer="16"/>
+<wire x1="40.64" y1="68.58" x2="40.64" y2="54.61" width="0.4064" layer="16"/>
+<wire x1="40.64" y1="54.61" x2="41.91" y2="53.34" width="0.4064" layer="16"/>
+<wire x1="41.91" y1="53.34" x2="48.77" y2="53.34" width="0.4064" layer="16"/>
+<wire x1="48.77" y1="53.34" x2="48.78" y2="53.33" width="0.4064" layer="16"/>
+<contactref element="1K" pad="1"/>
+<wire x1="46.99" y1="71.12" x2="46.99" y2="68.58" width="0.4064" layer="16"/>
+<wire x1="46.99" y1="68.58" x2="48.26" y2="67.31" width="0.4064" layer="16"/>
+<wire x1="48.26" y1="67.31" x2="58.42" y2="67.31" width="0.4064" layer="16"/>
+<wire x1="58.42" y1="67.31" x2="59.69" y2="68.58" width="0.4064" layer="16"/>
 </signal>
 <signal name="N$1">
@@
 <wire x1="71.12" y1="59.69" x2="73.66" y2="62.23" width="0.4064" layer="16"/>
 </signal>
+<signal name="N$3">
+<contactref element="POT_SIGNAL" pad="1"/>
+<contactref element="2K" pad="2"/>
+<wire x1="57.15" y1="76.2" x2="57.15" y2="73.66" width="0.4064" layer="16"/>
+<wire x1="57.15" y1="73.66" x2="54.61" y2="71.12" width="0.4064" layer="16"/>
+</signal>
 </signals>
