File: PCB/8266_DIYIOT_Board_O/Knob_8266.sch (EAGLE design)
At the start: 16 parts

Commit message: lots of updates
Parts:
- added 1K, 2K: (no value), eagle-ltspice:R0204/7
Connections:
- new net N$3: 2K.2, POT_SIGNAL.P
- net 5V: now also 1K.2
- net N$2: now also 1K.1, 2K.1; no longer POT_SIGNAL.P
Changed lines of the file:
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@@
 <layer number="97" name="Info" color="7" fill="1" visible="yes" active="yes"/>
 <layer number="98" name="Guide" color="6" fill="1" visible="yes" active="yes"/>
+<layer number="99" name="SpiceOrder" color="5" fill="1" visible="yes" active="yes"/>
 <layer number="101" name="Hidden" color="15" fill="1" visible="yes" active="yes"/>
 <layer number="102" name="Changes" color="12" fill="1" visible="yes" active="yes"/>
@@
 <part name="POT_SIGNAL" library="wirepad" deviceset="2,15/1,0" device=""/>
 <part name="5V_POT" library="wirepad" deviceset="2,15/1,0" device=""/>
+<part name="2K" library="eagle-ltspice" deviceset="R" device="0204/7"/>
+<part name="1K" library="eagle-ltspice" deviceset="R" device="0204/7"/>
 </parts>
 <sheets>
@@
 <instance part="POT_SIGNAL" gate="1" x="91.44" y="81.28"/>
 <instance part="5V_POT" gate="1" x="76.2" y="91.44"/>
+<instance part="2K" gate="G$1" x="81.28" y="73.66"/>
+<instance part="1K" gate="G$1" x="96.52" y="68.58"/>
 </instances>
 <busses>
@@
 <wire x1="127" y1="66.04" x2="127" y2="40.64" width="0.1524" layer="91"/>
 <wire x1="127" y1="40.64" x2="127" y2="38.1" width="0.1524" layer="91"/>
-<wire x1="127" y1="38.1" x2="106.68" y2="38.1" width="0.1524" layer="91"/>
+<wire x1="127" y1="38.1" x2="119.38" y2="38.1" width="0.1524" layer="91"/>
 <pinref part="U$4" gate="G$1" pin="GND"/>
+<wire x1="119.38" y1="38.1" x2="106.68" y2="38.1" width="0.1524" layer="91"/>
 <wire x1="127" y1="38.1" x2="139.7" y2="38.1" width="0.1524" layer="91"/>
 <junction x="127" y="38.1"/>
@@
 <pinref part="GND_1" gate="1" pin="P"/>
 <pinref part="GND_POT" gate="1" pin="P"/>
+<wire x1="101.6" y1="68.58" x2="119.38" y2="68.58" width="0.1524" layer="91"/>
+<wire x1="119.38" y1="68.58" x2="119.38" y2="38.1" width="0.1524" layer="91"/>
+<junction x="119.38" y="38.1"/>
+<junction x="101.6" y="68.58"/>
+<pinref part="1K" gate="G$1" pin="2"/>
 </segment>
 <segment>
@@
 <segment>
 <wire x1="76.2" y1="53.34" x2="73.66" y2="53.34" width="0.1524" layer="91"/>
-<wire x1="73.66" y1="53.34" x2="63.5" y2="53.34" width="0.1524" layer="91"/>
-<wire x1="63.5" y1="53.34" x2="63.5" y2="68.58" width="0.1524" layer="91"/>
-<wire x1="63.5" y1="68.58" x2="93.98" y2="68.58" width="0.1524" layer="91"/>
-<wire x1="93.98" y1="68.58" x2="93.98" y2="81.28" width="0.1524" layer="91"/>
+<wire x1="73.66" y1="53.34" x2="68.58" y2="53.34" width="0.1524" layer="91"/>
+<wire x1="68.58" y1="53.34" x2="68.58" y2="73.66" width="0.1524" layer="91"/>
 <pinref part="U$4" gate="G$1" pin="ADC"/>
 <junction x="73.66" y="53.34"/>
-<pinref part="POT_SIGNAL" gate="1" pin="P"/>
+<junction x="68.58" y="73.66"/>
+<wire x1="76.2" y1="73.66" x2="68.58" y2="73.66" width="0.1524" layer="91"/>
+<pinref part="2K" gate="G$1" pin="1"/>
+<junction x="76.2" y="73.66"/>
+<pinref part="1K" gate="G$1" pin="1"/>
+<junction x="91.44" y="68.58"/>
+<wire x1="91.44" y1="68.58" x2="76.2" y2="68.58" width="0.1524" layer="91"/>
+<junction x="76.2" y="68.58"/>
+<wire x1="76.2" y1="73.66" x2="76.2" y2="68.58" width="0.1524" layer="91"/>
 </segment>
 </net>
@@
 </segment>
 </net>
+<net name="N$3" class="0">
+<segment>
+<pinref part="POT_SIGNAL" gate="1" pin="P"/>
+<wire x1="93.98" y1="73.66" x2="93.98" y2="81.28" width="0.1524" layer="91"/>
+<wire x1="93.98" y1="73.66" x2="86.36" y2="73.66" width="0.1524" layer="91"/>
+<pinref part="2K" gate="G$1" pin="2"/>
+</segment>
+</net>
